File: minimal_max14906/minimal_max14906.kicad_pcb (KiCad board)
At the start: 4 copper layers, 70.8 x 50.2 mm, 114 parts, among them J10 TBP02R2-381-02BE, J11 TBP02R2-381-02BE, J12 CLP-102-02-G-D-BE, J13 CLP-108-02-G-D-BE, J14 CLP-108-02-G-D-BE, J15 CLP-102-02-G-D-BE, J2 TBP02R2-381-02BE, J3 TBP02R2-381-02BE, J4 CLP-102-02-G-D-BE, J5 CLP-102-02-G-D-BE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

Commit message: development backup
Parts:
- added MB1: mouse-bite-50mil-550mil, mouse_bite_footprints:mouse-bite-50mil-550mil, F.Cu at (118.1, 87.8)
- added MB6: mouse-bite-50mil-550mil, mouse_bite_footprints:mouse-bite-50mil-550mil, F.Cu at (152.4, 87.8)
- added MB8: mouse-bite-50mil-300mil, mouse_bite_footprints:mouse-bite-50mil-300mil, F.Cu at (151.8, 124.6)
- moved MB3 1.27 mm to (152.4, 99.6), turned to 90 degrees
- moved FID2 0.63 mm to (119.1, 115.4)
- moved MB2 0.63 mm to (117.5, 99.6), turned to -90 degrees
- moved MB4 0.63 mm to (117.5, 107.2), turned to -90 degrees
- moved MB5 0.63 mm to (153.0, 107.2), turned to 90 degrees
Connections:
- D4 pad 1: /SLED -> unconnected-(D4-Pad1)
- D5 pad 2: Net-(D4-Pad2) -> unconnected-(D5-Pad2)
Other:
- board size 70.8 x 50.2 mm -> 70.8 x 50.4 mm

Commit message: development backup
Connections:
- D4 pad 1: unconnected-(D4-Pad1) -> /SLED
- D5 pad 2: unconnected-(D5-Pad2) -> Net-(D4-Pad2)
- TP31 pad 1: /FIELD_POWER_DETECTED_ISO -> /VDD_OK_ISO
- TP32 pad 1: /VDD_OK_ISO -> /FIELD_POWER_DETECTED_ISO
Routing:
- net /VDD_OK_ISO: track 28.0 -> 7.60 mm
- net /FIELD_POWER_DETECTED_ISO: track 7.75 -> 27.7 mm
- net /FIELD_POWER_DETECTED: track 38.0 -> 36.9 mm
- net /VDD_OK: track 35.4 -> 34.6 mm
- net /SYNCH: track 17.7 -> 17.1 mm
- net /~{CS_ISO}: track 16.0 -> 15.5 mm
- net /SDO_ISO: track 15.4 -> 14.9 mm
Other:
- outline, holes or cut-outs redrawn

Commit message: development backup
Parts:
- J13, J14: value CLP-108-02-G-D-BE -> CLP-109-02-G-D-BE; footprint connector_footprints:CLP-108-02-G-D-BE -> connector_footprints:CLP-109-02-G-D-BE
- moved FID1 16.3 mm to (119.1, 97.5)
- moved FID3 16.3 mm to (151.4, 97.5)
- moved J10 2.54 mm to (101.3, 112.1)
- moved J11 2.54 mm to (169.2, 112.1)
- moved J2 2.54 mm to (101.3, 94.8)
- moved J3 2.54 mm to (169.2, 94.8)
- moved J13 0.64 mm to (113.7, 87.8)
- moved J14 0.64 mm to (156.8, 87.8)
Connections:
- J13 pad 1: /D3_ISO -> /FIELD_POWER_DETECTED_ISO
- J13 pad 11: /SDI_ISO -> /CLK_ISO
- J13 pad 13: /3V3_ISO -> /SDI_ISO
- J13 pad 15: GND -> /3V3_ISO
- J13 pad 3: /D4_ISO -> /D3_ISO
- J13 pad 5: /SDO_ISO -> /D4_ISO
- J13 pad 7: /~{CS_ISO} -> /SDO_ISO
- J13 pad 9: /CLK_ISO -> /~{CS_ISO}
Routing:
- net /VDD_OK_ISO: track 7.60 -> 10.2 mm
- net /FIELD_POWER_DETECTED_ISO: track 27.7 -> 30.3 mm
Other:
- board size 70.8 x 50.4 mm -> 75.8 x 50.4 mm

Commit message: development backup
Parts:
- added MB7: mouse-bite-50mil-200mil, mouse_bite_footprints:mouse-bite-50mil-200mil, F.Cu at (153.0, 121.5)
- MB8: value mouse-bite-50mil-300mil -> mouse-bite-50mil-200mil; footprint mouse_bite_footprints:mouse-bite-50mil-300mil -> mouse_bite_footprints:mouse-bite-50mil-200mil
- moved MB8 18.3 mm to (133.7, 121.5), turned to 90 degrees
- moved J15 17.9 mm to (131.2, 121.5), turned to 0 degrees
- moved TP28 17.0 mm to (134.4, 122.1), turned to 0 degrees
- moved TP27 16.0 mm to (134.4, 120.8), turned to 0 degrees
- moved S1 8.60 mm to (143.4, 119.6)
- moved J12 6.35 mm to (155.6, 121.5), turned to 180 degrees
- moved TP29 4.02 mm to (152.4, 120.8), turned to 180 degrees
- moved TP21 2.54 mm to (155.6, 107.9)
- moved TP22 2.54 mm to (155.6, 106.6)
- moved J4 2.54 mm to (111.1, 99.6)
- moved J7 2.54 mm to (111.1, 107.2)
- moved TP19 2.54 mm to (114.9, 106.6)
- moved TP20 2.54 mm to (114.9, 107.9)
- moved J5 2.54 mm to (159.4, 99.6)
- moved J8 2.54 mm to (159.4, 107.2)
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Routing:
- net /INT_VIN: track 8.43 -> 14.1 mm
- added copper zone on In1.Cu, net /EXT_VIN
- added copper zone on In1.Cu, net /INT_VIN
Other:
- board size 75.8 x 50.4 mm -> 75.8 x 45.1 mm
