File: minimal_max14906/minimal_max14906.kicad_sch (KiCad schematic)
At the start: 104 parts, among them J10 TBP02R2-381-02BE, J11 TBP02R2-381-02BE, J12 CLP-103-02-G-D-BE, J13 CLP-108-02-G-D-BE, J14 CLP-108-02-G-D-BE, J2 TBP02R2-381-02BE, J3 TBP02R2-381-02BE, J4 CLP-102-02-G-D-BE, J5 CLP-102-02-G-D-BE, J6 CLP-102-02-G-D-BE, J7 CLP-102-02-G-D-BE, J8 CLP-102-02-G-D-BE, J9 CLP-102-02-G-D-BE, Q1 -60.0 V, Q2 -60.0 V, Q3 -60.0 V, Q4 -60.0 V, Q5 100 V, U1 ADUM1252AUA+, U2 MAX22441CAEE+, U3 MAX22442CAEE+, U4 ADUM1252AUA+, U5 MAX14906ATM+

Commit message: development backup
Connections:
- net 3V3_ISO: now also J13.13, J14.3, TP2.1; no longer J13.3, J14.13, TP25.1
- net CLK_ISO: now also J13.5, TP5.1; no longer J13.9, TP6.1
- net D1_ISO: now also J14.5, TP8.1; no longer J14.1, TP12.1
- net D2_ISO: now also J14.7, TP9.1; no longer J14.3, TP13.1
- net D3_ISO: now also J13.9, TP6.1; no longer J13.13, TP2.1
- net D4_ISO: now also J13.11, TP7.1; no longer J13.15, TP3.1
- net EN_ISO: now also J14.9, TP11.1; no longer J14.5, TP10.1
- net GND: now also J13.15, J14.1, TP3.1; no longer J13.1, J14.15, TP26.1
- net SDI_ISO: now also J13.7, TP4.1; no longer J13.11, TP7.1
- net SDO_ISO: now also J13.3, TP25.1; no longer J13.7, TP4.1
- net SYNCH_ISO: now also J14.11, TP10.1; no longer J14.7, TP11.1
- net ~{CS_ISO}: now also J13.1, TP26.1; no longer J13.5, TP5.1
- net ~{FAULT_ISO}: now also J14.13, TP13.1; no longer J14.9, TP9.1
- net ~{READY_ISO}: now also J14.15, TP12.1; no longer J14.11, TP8.1
Other:
- moved on the sheet: J14
Changed lines of the file:
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@@
 	)
 	(junction
-		(at 48.26 152.4)
-		(diameter 0)
-		(color 0 0 0 0)
-	)
-	(junction
 		(at 97.79 99.06)
 		(diameter 0)
@@
 	)
 	(junction
+		(at 48.26 170.18)
+		(diameter 0)
+		(color 0 0 0 0)
+	)
+	(junction
 		(at 266.7 157.48)
 		(diameter 0)
@@
 	(wire
 		(pts
+			(xy 48.26 170.18) (xy 48.26 171.45)
+		)
+		(stroke
+			(width 0)
+			(type default)
+		)
+	)
+	(wire
+		(pts
 			(xy 133.35 88.9) (xy 146.05 88.9)
 		)
@@
 	(wire
 		(pts
-			(xy 48.26 152.4) (xy 60.96 152.4)
+			(xy 45.72 152.4) (xy 60.96 152.4)
 		)
 		(stroke
@@
 	(wire
 		(pts
-			(xy 48.26 152.4) (xy 45.72 152.4)
-		)
-		(stroke
-			(width 0)
-			(type default)
-		)
-	)
-	(wire
-		(pts
 			(xy 321.31 119.38) (xy 342.9 119.38)
 		)
@@
 	(wire
 		(pts
-			(xy 48.26 171.45) (xy 48.26 152.4)
-		)
-		(stroke
-			(width 0)
-			(type default)
-		)
-	)
-	(wire
-		(pts
 			(xy 210.82 81.28) (xy 210.82 86.36)
 		)
@@
 	(wire
 		(pts
-			(xy 45.72 170.18) (xy 60.96 170.18)
+			(xy 45.72 170.18) (xy 48.26 170.18)
 		)
 		(stroke
@@
 	(wire
 		(pts
+			(xy 48.26 170.18) (xy 60.96 170.18)
+		)
+		(stroke
+			(width 0)
+			(type default)
+		)
+	)
+	(wire
+		(pts
 			(xy 125.73 109.22) (xy 148.59 109.22)
 		)
@@
 	)
 	(label "D2_ISO"
-		(at 50.8 189.23 0)
+		(at 50.8 196.85 0)
 		(effects
 			(font
@@
 	)
 	(label "~{FAULT_ISO}"
-		(at 50.8 196.85 0)
+		(at 50.8 189.23 0)
 		(effects
 			(font
@@
 	)
 	(label "D3_ISO"
-		(at 50.8 167.64 0)
+		(at 50.8 162.56 0)
 		(effects
 			(font
@@
 	)
 	(label "~{READY_ISO}"
-		(at 50.8 199.39 0)
+		(at 50.8 186.69 0)
 		(effects
 			(font
@@
 	)
 	(label "SDI_ISO"
-		(at 50.8 165.1 0)
+		(at 50.8 160.02 0)
 		(effects
 			(font
@@
 	)
 	(label "SYNCH_ISO"
-		(at 50.8 194.31 0)
+		(at 50.8 191.77 0)
 		(effects
 			(font
@@
 	)
 	(label "D4_ISO"
-		(at 50.8 170.18 0)
+		(at 50.8 165.1 0)
 		(effects
 			(font
@@
 	)
 	(label "SDO_ISO"
-		(at 50.8 160.02 0)
+		(at 50.8 154.94 0)
 		(effects
 			(font
@@
 	)
 	(label "D1_ISO"
-		(at 50.8 186.69 0)
+		(at 50.8 199.39 0)
 		(effects
 			(font
@@
 	)
 	(label "~{CS_ISO}"
-		(at 50.8 157.48 0)
+		(at 50.8 152.4 0)
 		(effects
 			(font
@@
 	)
 	(label "EN_ISO"
-		(at 50.8 191.77 0)
+		(at 50.8 194.31 0)
 		(effects
 			(font
@@
 	)
 	(label "CLK_ISO"
-		(at 50.8 162.56 0)
+		(at 50.8 157.48 0)
 		(effects
 			(font
@@
 	)
 	(label "3V3_ISO"
-		(at 50.8 154.94 0)
+		(at 50.8 167.64 0)
 		(effects
 			(font
@@
 	(symbol
 		(lib_id "UNITED_CONNECTORS_DATA_BASE:J_CLP-108-02-G-D-BE")
-		(at 40.64 195.58 0)
-		(mirror y)
+		(at 40.64 195.58 180)
 		(unit 1)
 		(exclude_from_sim no)
@@
 		)
 		(property "Footprint" "connector_footprints:CLP-108-02-G-D-BE"
-			(at 35.56 210.82 0)
+			(at 35.56 180.34 0)
 			(show_name yes)
 			(effects
@@
 		)
 		(property "Datasheet" "https://suddendocs.samtec.com/catalog_english/clp_sm.pdf?_gl=1*1y4jlr9*_gcl_au*MTM0MTYyNTQ5MS4xNzM2MDk5MTUz*_ga*MTYxNDYyMTQ0Mi4xNzM2MDk5MTUz*_ga_3KFNZC07WW*MTczNjY4MDQ4OS4xNS4xLjE3MzY2ODEzNzcuNjAuMC4w"
-			(at 35.56 213.36 0)
+			(at 35.56 177.8 0)
 			(show_name yes)
 			(effects
@@
 		)
 		(property "Description" "Samtec CLP-1xx-02-G-D-BE series,  8 positions connector,  1.27 mm pitch,  Black,  Vertical mounting,  5.2 A,  300 V,  Surface Mount,  Tin plated"
-			(at 35.56 215.9 0)
+			(at 35.56 175.26 0)
 			(show_name yes)
 			(effects
@@
 		)
 		(property "Color" "Black"
-			(at 35.56 218.44 0)
+			(at 35.56 172.72 0)
 			(show_name yes)
 			(effects
@@
 		)
 		(property "Contact Plating" "Tin"
-			(at 35.56 220.98 0)
+			(at 35.56 170.18 0)
 			(show_name yes)
 			(effects
@@
 		)
 		(property "Current Rating (A)" "5.2"
-			(at 35.56 223.52 0)
+			(at 35.56 167.64 0)
 			(show_name yes)
 			(effects
@@
 		)
 		(property "MPN" "CLP-108-02-G-D-BE"
-			(at 35.56 226.06 0)
+			(at 35.56 165.1 0)
 			(show_name yes)
 			(effects
@@
 		)
 		(property "Manufacturer" "Samtec"
-			(at 35.56 228.6 0)
+			(at 35.56 162.56 0)
 			(show_name yes)
 			(effects
@@
 		)
 		(property "Mounting Angle" "Vertical"
-			(at 35.56 231.14 0)
+			(at 35.56 160.02 0)
 			(show_name yes)
 			(effects
@@
 		)
 		(property "Mounting Style" "Surface Mount"
-			(at 35.56 233.68 0)
+			(at 35.56 157.48 0)
 			(show_name yes)
 			(effects
@@
 		)
 		(property "Number of Rows" "2"
-			(at 35.56 236.22 0)
+			(at 35.56 154.94 0)
 			(show_name yes)
 			(effects
@@
 		)
 		(property "Pin Count" "8"
-			(at 35.56 238.76 0)
+			(at 35.56 152.4 0)
 			(show_name yes)
 			(effects
@@
 		)
 		(property "Pitch (mm)" "1.27"
-			(at 35.56 241.3 0)
+			(at 35.56 149.86 0)
 			(show_name yes)
 			(effects
@@
 		)
 		(property "Series" "CLP-1xx-02-G-D-BE"
-			(at 35.56 243.84 0)
+			(at 35.56 147.32 0)
 			(show_name yes)
 			(effects
@@
 		)
 		(property "Symbol Name" "J_CLP-108-02-G-D-BE"
-			(at 35.56 246.38 0)
+			(at 35.56 144.78 0)
 			(show_name yes)
 			(effects
@@
 		)
 		(property "Trustedparts Search" "https://www.trustedparts.com/en/search/CLP-108-02-G-D-BE"
-			(at 35.56 248.92 0)
+			(at 35.56 142.24 0)
 			(show_name yes)
 			(effects
@@
 		)
 		(property "Voltage Rating (V)" "300"
-			(at 35.56 251.46 0)
+			(at 35.56 139.7 0)
 			(show_name yes)
 			(effects

Commit message: development backup
Parts:
- removed J9: CLP-102-02-G-D-BE, connector_footprints:CLP-102-02-G-D-BE, symbol UNITED_CONNECTORS_DATA_BASE:J_CLP-102-02-G-D-BE
- removed MB6: mouse-bite-midle-50mil-200mil, mouse_bite_footprints:mouse-bite-midle-50mil-200mil, symbol UNITED_MOUSE_BITES_DATA_BASE:mouse-bite-midle-50mil-200mil
- removed TP23, TP24: TestPoint, test_point_footprints:TestPoint_THTPad_Castelated, symbol UNITED_TEST_POINTS:TestPoint_Castelated
- added C30, C33: 100 nF, capacitor_footprints:C_0402_1005Metric, symbol UNITED_CAPACITORS_DATA_BASE:C_GCM155R71H104KE02D
- added C31, C32: 1 nF, capacitor_footprints:C_0402_1005Metric, symbol UNITED_CAPACITORS_DATA_BASE:C_GCM155R71H102KA37D
- added J15: CLP-102-02-G-D-BE, connector_footprints:CLP-102-02-G-D-BE, symbol UNITED_CONNECTORS_DATA_BASE:J_CLP-102-02-G-D-BE
- added Q6: 100 V, transistor_footprints:SOT-323, symbol UNITED_TRANSISTORS_DATA_BASE:Q_BSS123WQ-7-F
- added R9: 10 kΩ, resistor_footprints:R_0402_1005Metric, symbol UNITED_RESISTORS_DATA_BASE:R_ERJ-2RKF1002X
- added TP27, TP28, TP29, TP30, TP31, TP32: TestPoint, test_point_footprints:TestPoint_THTPad_Castelated, symbol UNITED_TEST_POINTS:TestPoint_Castelated
- added U6: ADUM1252AUA+, analog_devices_footprints:21-0036_ADI, symbol UNITED_IC_ADI:U_ADUM1252AUA+
- J12: value CLP-103-02-G-D-BE -> CLP-102-02-G-D-BE; footprint connector_footprints:CLP-103-02-G-D-BE -> connector_footprints:CLP-102-02-G-D-BE; symbol UNITED_CONNECTORS_DATA_BASE:J_CLP-103-02-G-D-BE -> UNITED_CONNECTORS_DATA_BASE:J_CLP-102-02-G-D-BE; MPN CLP-103-02-G-D-BE -> CLP-102-02-G-D-BE; Pin Count 3 -> 2; Symbol Name J_CLP-103-02-G-D-BE -> J_CLP-102-02-G-D-BE; Trustedparts Search https://www.trustedparts.com/en/search/CLP-103-02-G-D-BE -> https://www.trustedparts.com/en/search/CLP-102-02-G-D-BE
- MB2, MB3, MB4, MB5: value mouse-bite-midle-50mil-200mil -> mouse-bite-50mil-200mil; footprint mouse_bite_footprints:mouse-bite-midle-50mil-200mil -> mouse_bite_footprints:mouse-bite-50mil-200mil; symbol UNITED_MOUSE_BITES_DATA_BASE:mouse-bite-midle-50mil-200mil -> UNITED_MOUSE_BITES_DATA_BASE:mouse-bite-50mil-200mil
Connections:
- net 3V3_EXT is gone; now on net 3V3: R8.1
- net 3V3: now also C32.1, C33.1, R9.1, U6.8 (VDD2)
- net 3V3_ISO: now also C30.1, C31.1, U6.1 (VDD1)
- net CLK_ISO: now also J13.9, TP6.1; no longer J13.5, TP5.1
- net D1_ISO: now also J14.15, TP12.1; no longer J14.5, TP8.1
- net D2_ISO: now also J14.13, TP13.1; no longer J14.7, TP9.1
- net D3_ISO: now also J13.1, TP25.1; no longer J13.9, TP6.1
- net D4_ISO: now also J13.3, TP26.1; no longer J13.11, TP7.1
- net EXT_VIN: now also J12.2, J12.4, TP29.1; no longer J12.5, J12.6
- net FIELD_POWER_DETECTED: now also U6.6 (SCL2)
- net GND: now also C30.2, C31.2, U6.4 (GND1)
- net GNDA: now also J12.1, C32.2, C33.2, J15.2, J15.4, Q6.2 (S), TP28.1, TP30.1, U6.5 (GND2); no longer J12.4
- net INT_VIN: now also J15.1, J15.3, TP27.1; no longer J12.1, J12.2
- net SDI_ISO: now also J13.11, TP7.1; no longer J13.7, TP4.1
- net SDO_ISO: now also J13.5, TP5.1; no longer J13.3, TP25.1
- net ~{CS_ISO}: now also J13.7, TP4.1; no longer J13.1, TP26.1
- net ~{FAULT_ISO}: now also J14.7, TP9.1; no longer J14.13, TP13.1
- net ~{READY_ISO}: now also J14.5, TP8.1; no longer J14.15, TP12.1
- net VDD_OK_GATE: now reaches D3.2, R1.2
- net VDD_OK_GATE: now also Q6.1 (G)
- new net FIELD_POWER_DETECTED_ISO: TP31.1, U6.3 (SCL1)
- new net VDD_OK: Q6.3 (D), R9.2, U6.7 (SDA2)
- new net VDD_OK_ISO: TP32.1, U6.2 (SDA1)
Other:
- moved on the sheet: Q5, R6, R7, R8, S1, TP15, TP16, TP17, TP18, TP19, TP20, TP21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

Commit message: development backup
Parts:
- added MB1, MB6: mouse-bite-50mil-550mil, mouse_bite_footprints:mouse-bite-50mil-550mil, symbol UNITED_MOUSE_BITES_DATA_BASE:mouse-bite-50mil-550mil
- added MB8: mouse-bite-50mil-300mil, mouse_bite_footprints:mouse-bite-50mil-300mil, symbol UNITED_MOUSE_BITES_DATA_BASE:mouse-bite-50mil-300mil
Connections:
- net SLED: no longer D4.1
- net at D4.2, R2.1: no longer D5.2
Other:
- moved on the sheet: C1, C10, C11, C12, C13, C14, C15, C16, C2, C3, C4, C5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

Commit message: development backup
Connections:
- net FIELD_POWER_DETECTED_ISO: now also TP32.1; no longer TP31.1
- net SLED: now also D4.1
- net VDD_OK_ISO: now also TP31.1; no longer TP32.1
- net at D4.2, R2.1: now also D5.2
Other:
- moved on the sheet: D4, TP31, TP32
Changed lines of the file:
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@@
 	)
 	(junction
-		(at 96.52 240.03)
-		(diameter 0)
-		(color 0 0 0 0)
-	)
-	(junction
 		(at 215.9 196.85)
 		(diameter 0)
@@
 	)
 	(junction
+		(at 96.52 243.84)
+		(diameter 0)
+		(color 0 0 0 0)
+	)
+	(junction
 		(at 308.61 119.38)
 		(diameter 0)
@@
 	(wire
 		(pts
-			(xy 96.52 240.03) (xy 96.52 242.57)
+			(xy 96.52 228.6) (xy 96.52 243.84)
 		)
 		(stroke
@@
 	(wire
 		(pts
-			(xy 96.52 228.6) (xy 96.52 240.03)
-		)
-		(stroke
-			(width 0)
-			(type default)
-		)
-	)
-	(wire
-		(pts
 			(xy 45.72 209.55) (xy 60.96 209.55)
 		)
@@
 	(symbol
 		(lib_id "UNITED_DIODES_DATA_BASE:D_APHHS1005CGCK")
-		(at 96.52 245.11 90)
+		(at 96.52 250.19 90)
 		(mirror x)
 		(unit 1)
@@
 		(on_board yes)
 		(dnp no)
+		(fields_autoplaced yes)
 		(property "Reference" "D4"
 			(at 100.33 251.8409 90)
@@
 		)
 		(property "Value" "1.8 V"
-			(at 97.79 249.174 0)
+			(at 97.79 254.254 0)
 			(effects
 				(font
@@
 		)
 		(property "Footprint" "diode_footprints:LED_GREEN_0402_1005Metric"
-			(at 104.14 245.11 0)
+			(at 104.14 250.19 0)
 			(show_name yes)
 			(effects
@@
 		)
 		(property "Datasheet" "https://www.kingbrightusa.com/product.asp?catalog_name=LED&product_id=APHHS1005CGCK"
-			(at 106.68 245.11 0)
+			(at 106.68 250.19 0)
 			(show_name yes)
 			(effects
@@
 		)
 		(property "Description" "Green LED SMD 1.8 V"
-			(at 109.22 245.11 0)
+			(at 109.22 250.19 0)
 			(show_name yes)
 			(effects
@@
 		)
 		(property "Diode Type" "Green LED"
-			(at 111.76 245.11 0)
+			(at 111.76 250.19 0)
 			(effects
 				(font
@@
 		)
 		(property "MPN" "APHHS1005CGCK"
-			(at 114.3 245.11 0)
+			(at 114.3 250.19 0)
 			(effects
 				(font
@@
 		)
 		(property "Manufacturer" "Kingbright"
-			(at 116.84 245.11 0)
+			(at 116.84 250.19 0)
 			(effects
 				(font
@@
 		)
 		(property "Maximum DC Current (A)" "0.03"
-			(at 119.38 245.11 0)
+			(at 119.38 250.19 0)
 			(effects
 				(font
@@
 		)
 		(property "Series" "APHHS1005CGCK"
-			(at 121.92 245.11 0)
+			(at 121.92 250.19 0)
 			(effects
 				(font
@@
 		)
 		(property "Symbol Name" "D_APHHS1005CGCK"
-			(at 124.46 245.11 0)
+			(at 124.46 250.19 0)
 			(effects
 				(font
@@
 		)
 		(property "Trustedparts Search" "https://www.trustedparts.com/en/search/APHHS1005CGCK"
-			(at 127 245.11 0)
+			(at 127 250.19 0)
 			(effects
 				(font
@@
 	(symbol
 		(lib_id "UNITED_TEST_POINTS:TestPoint_Castelated")
-		(at 59.69 35.56 90)
+		(at 59.69 38.1 90)
 		(mirror x)
 		(unit 1)
@@
 		(fields_autoplaced yes)
 		(property "Reference" "TP32"
-			(at 54.61 35.5599 90)
+			(at 54.61 38.0999 90)
 			(effects
 				(font
@@
 		)
 		(property "Value" "TestPoint"
-			(at 57.15 38.1 0)
+			(at 57.15 40.64 0)
 			(effects
 				(font
@@
 		)
 		(property "Footprint" "test_point_footprints:TestPoint_THTPad_Castelated"
-			(at 64.77 38.1 0)
+			(at 64.77 40.64 0)
 			(effects
 				(font
@@
 		)
 		(property "Datasheet" "~"
-			(at 59.69 38.1 0)
+			(at 59.69 40.64 0)
 			(effects
 				(font
@@
 		)
 		(property "Description" "test point"
-			(at 62.23 38.1 0)
+			(at 62.23 40.64 0)
 			(effects
 				(font
@@
 	(symbol
 		(lib_id "UNITED_TEST_POINTS:TestPoint_Castelated")
-		(at 59.69 38.1 90)
+		(at 59.69 35.56 90)
 		(mirror x)
 		(unit 1)
@@
 		(fields_autoplaced yes)
 		(property "Reference" "TP31"
-			(at 54.61 38.0999 90)
+			(at 54.61 35.5599 90)
 			(effects
 				(font
@@
 		)
 		(property "Value" "TestPoint"
-			(at 57.15 40.64 0)
+			(at 57.15 38.1 0)
 			(effects
 				(font
@@
 		)
 		(property "Footprint" "test_point_footprints:TestPoint_THTPad_Castelated"
-			(at 64.77 40.64 0)
+			(at 64.77 38.1 0)
 			(effects
 				(font
@@
 		)
 		(property "Datasheet" "~"
-			(at 59.69 40.64 0)
+			(at 59.69 38.1 0)
 			(effects
 				(font
@@
 		)
 		(property "Description" "test point"
-			(at 62.23 40.64 0)
+			(at 62.23 38.1 0)
 			(effects
 				(font

Commit message: development backup
Parts:
- J13, J14: value CLP-108-02-G-D-BE -> CLP-109-02-G-D-BE; footprint connector_footprints:CLP-108-02-G-D-BE -> connector_footprints:CLP-109-02-G-D-BE; symbol UNITED_CONNECTORS_DATA_BASE:J_CLP-108-02-G-D-BE -> UNITED_CONNECTORS_DATA_BASE:J_CLP-109-02-G-D-BE; MPN CLP-108-02-G-D-BE -> CLP-109-02-G-D-BE; Pin Count 8 -> 9; Symbol Name J_CLP-108-02-G-D-BE -> J_CLP-109-02-G-D-BE; Trustedparts Search https://www.trustedparts.com/en/search/CLP-108-02-G-D-BE -> https://www.trustedparts.com/en/search/CLP-109-02-G-D-BE
Connections:
- net 3V3_ISO: now also J13.15; no longer J13.13
- net CLK_ISO: now also J13.11; no longer J13.9
- net D3_ISO: now also J13.3; no longer J13.1
- net D4_ISO: now also J13.5; no longer J13.3
- net FIELD_POWER_DETECTED_ISO: now also J13.1
- net GND: now also J13.17, J13.18, J14.18; no longer J13.15
- net SDI_ISO: now also J13.13; no longer J13.11
- net SDO_ISO: now also J13.7; no longer J13.5
- net VDD_OK_ISO: now also J14.17
- net ~{CS_ISO}: now also J13.9; no longer J13.7
Other:
- moved on the sheet: TP31, TP32

Commit message: development backup
Parts:
- removed MB8: mouse-bite-50mil-300mil, mouse_bite_footprints:mouse-bite-50mil-300mil, symbol UNITED_MOUSE_BITES_DATA_BASE:mouse-bite-50mil-300mil
- added MB7, MB8: mouse-bite-50mil-200mil, mouse_bite_footprints:mouse-bite-50mil-200mil, symbol UNITED_MOUSE_BITES_DATA_BASE:mouse-bite-50mil-200mil
Changed lines of the file:
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@@
 	)
 	(symbol
-		(lib_id "UNITED_MOUSE_BITES_DATA_BASE:mouse-bite-50mil-300mil")
-		(at 104.14 71.12 90)
-		(unit 1)
-		(exclude_from_sim no)
-		(in_bom yes)
-		(on_board yes)
-		(dnp no)
-		(fields_autoplaced yes)
-		(property "Reference" "MB8"
-			(at 96.52 71.12 0)
-			(effects
-				(font
-					(size 1.27 1.27)
-				)
-				(justify left)
-				(hide yes)
-			)
-		)
-		(property "Value" "mouse-bite-50mil-300mil"
-			(at 111.76 71.12 0)
-			(effects
-				(font
-					(size 1.27 1.27)
-				)
-				(justify left)
-				(hide yes)
-			)
-		)
-		(property "Footprint" "mouse_bite_footprints:mouse-bite-50mil-300mil"
-			(at 109.22 71.12 0)
-			(effects
-				(font
-					(size 1.27 1.27)
-				)
-				(justify left)
-				(hide yes)
-			)
-		)
-		(property "Datasheet" ""
-			(at 104.14 71.12 0)
-			(effects
-				(font
-					(size 1.27 1.27)
-				)
-				(hide yes)
-			)
-		)
-		(property "Description" ""
-			(at 104.14 71.12 0)
-			(effects
-				(font
-					(size 1.27 1.27)
-				)
-				(hide yes)
-			)
-		)
-		(instances
-			(project "minimal_max14906"
-				(path "/0138bc01-efaa-4f20-bf65-043bbc1a8346"
-					(reference "MB8")
-					(unit 1)
-				)
-			)
-		)
-	)
-	(symbol
 		(lib_id "UNITED_IC_ADI:U_MAX14906ATM+")
 		(at 215.9 152.4 0)
@@
 	)
 	(symbol
+		(lib_id "UNITED_MOUSE_BITES_DATA_BASE:mouse-bite-50mil-200mil")
+		(at 153.67 82.55 0)
+		(unit 1)
+		(exclude_from_sim no)
+		(in_bom yes)
+		(on_board yes)
+		(dnp no)
+		(fields_autoplaced yes)
+		(property "Reference" "MB8"
+			(at 153.67 74.93 0)
+			(effects
+				(font
+					(size 1.27 1.27)
+				)
+				(justify left)
+				(hide yes)
+			)
+		)
+		(property "Value" "mouse-bite-50mil-200mil"
+			(at 153.67 90.17 0)
+			(effects
+				(font
+					(size 1.27 1.27)
+				)
+				(justify left)
+				(hide yes)
+			)
+		)
+		(property "Footprint" "mouse_bite_footprints:mouse-bite-50mil-200mil"
+			(at 153.67 87.63 0)
+			(effects
+				(font
+					(size 1.27 1.27)
+				)
+				(justify left)
+				(hide yes)
+			)
+		)
+		(property "Datasheet" ""
+			(at 153.67 82.55 0)
+			(effects
+				(font
+					(size 1.27 1.27)
+				)
+				(hide yes)
+			)
+		)
+		(property "Description" ""
+			(at 153.67 82.55 0)
+			(effects
+				(font
+					(size 1.27 1.27)
+				)
+				(hide yes)
+			)
+		)
+		(instances
+			(project "minimal_max14906"
+				(path "/0138bc01-efaa-4f20-bf65-043bbc1a8346"
+					(reference "MB8")
+					(unit 1)
+				)
+			)
+		)
+	)
+	(symbol
 		(lib_id "UNITED_CAPACITORS_DATA_BASE:C_GCM155R71H104KE02D")
 		(at 85.09 104.14 90)
@@
 					(unit 1)
 				)
+			)
+		)
+	)
+	(symbol
+		(lib_id "UNITED_MOUSE_BITES_DATA_BASE:mouse-bite-50mil-200mil")
+		(at 153.67 59.69 0)
+		(unit 1)
+		(exclude_from_sim no)
+		(in_bom yes)
+		(on_board yes)
+		(dnp no)
+		(fields_autoplaced yes)
+		(property "Reference" "MB7"
+			(at 153.67 52.07 0)
+			(effects
+				(font
+					(size 1.27 1.27)
+				)
+				(justify left)
+				(hide yes)
+			)
+		)
+		(property "Value" "mouse-bite-50mil-200mil"
+			(at 153.67 67.31 0)
+			(effects
+				(font
+					(size 1.27 1.27)
+				)
+				(justify left)
+				(hide yes)
+			)
+		)
+		(property "Footprint" "mouse_bite_footprints:mouse-bite-50mil-200mil"
+			(at 153.67 64.77 0)
+			(effects
+				(font
+					(size 1.27 1.27)
+				)
+				(justify left)
+				(hide yes)
+			)
+		)
+		(property "Datasheet" ""
+			(at 153.67 59.69 0)
+			(effects
+				(font
+					(size 1.27 1.27)
+				)
+				(hide yes)
+			)
+		)
+		(property "Description" ""
+			(at 153.67 59.69 0)
+			(effects
+				(font
+					(size 1.27 1.27)
+				)
+				(hide yes)
+			)
+		)
+		(instances
+			(project "minimal_max14906"
+				(path "/0138bc01-efaa-4f20-bf65-043bbc1a8346"
+					(reference "MB7")
+					(unit 1)
+				)

Commit message: development backup
Parts:
- removed J10, J11, J2, J3: TBP02R2-381-02BE, connector_footprints:TBP02R2-381-02BE, symbol UNITED_CONNECTORS_DATA_BASE:J_TBP02R2-381-02BE
- renumbered C3 to C1, C5 to C10, C15 to C12, C17 to C13, C27 to C14, C2 to C15, C6 to C16, C12 to C17, C16 to C18, C18 to C19, C7 to C2, C28 to C20, C29 to C21, C4 to C22, C8 to C23, C10 to C24, C14 to C25, C22 to C26, C24 to C27, C20 to C28, C26 to C29, C9 to C3, C13 to C4, C19 to C5, C25 to C6, C21 to C7, C23 to C8, C1 to C9, D5 to D1, D4 to D2, D7 to D3, D6 to D4, D9 to D5, D8 to D6, D3 to D7, D11 to D8, D10 to D9, J13 to J1, J4 to J2, J7 to J3, J6 to J4, J15 to J5, J12 to J6, J14 to J7, J5 to J8, J8 to J9, MB4 to MB3, MB8 to MB4, MB7 to MB5, MB3 to MB7, MB5 to MB8, Q3 to Q2, Q6 to Q3, Q5 to Q4, Q2 to Q5, Q4 to Q6, R2 to R1, R3 to R2, R1 to R3, R9 to R6, R8 to R7, R6 to R8, R7 to R9, TP32 to TP1, TP16 to TP10, TP15 to TP11, TP19 to TP12, TP20 to TP13, TP27 to TP14, TP28 to TP15, TP29 to TP16, TP30 to TP17, TP31 to TP18, TP12 to TP19, TP25 to TP2, TP13 to TP20, TP10 to TP21, TP11 to TP22, TP9 to TP23, TP8 to TP24, TP1 to TP25, TP14 to TP26, TP17 to TP27, TP18 to TP28, TP22 to TP29, TP26 to TP3, TP21 to TP30, TP5 to TP4, TP4 to TP5, TP2 to TP8, TP3 to TP9, U5 to U3, U3 to U4, U4 to U5
Other:
- moved on the sheet: J2, J3, J8, J9, TP10, TP11, TP12, TP13, TP27, TP28, TP29, TP30

Commit message: development backup
Connections:
- net 3V3_ISO: now also J1.4, J7.16; no longer J1.15, J7.3
- net CHANNEL_2: now also J8.3, J8.4; no longer J8.1, J8.2
- net CHANNEL_4: now also J3.3, J3.4; no longer J3.1, J3.2
- net CLK_ISO: now also J1.8; no longer J1.11
- net D1_ISO: now also J7.4; no longer J7.15
- net D2_ISO: now also J7.6; no longer J7.13
- net D3_ISO: now also J1.16; no longer J1.3
- net D4_ISO: now also J1.14; no longer J1.5
- net EN_ISO: now also J7.10; no longer J7.9
- net FIELD_POWER_DETECTED_ISO: now also J1.18; no longer J1.1
- net GND: now also J1.1, J1.11, J1.13, J1.15, J1.3, J1.5, J1.7, J1.9, J7.11, J7.13, J7.15, J7.17, J7.3, J7.5, J7.7, J7.9; no longer J1.10, J1.12, J1.14, J1.16, J1.18, J1.4, J1.6, J1.8, J7.10, J7.12, J7.14, J7.16, J7.2, J7.4, J7.6, J7.8
- net GNDA: now also J3.1, J3.2, J8.1, J8.2; no longer J3.3, J3.4, J8.3, J8.4
- net SDI_ISO: now also J1.6; no longer J1.13
- net SDO_ISO: now also J1.12; no longer J1.7
- net SYNCH_ISO: now also J7.8; no longer J7.11
- net VDD_OK_ISO: now also J7.2; no longer J7.17
- net ~{CS_ISO}: now also J1.10; no longer J1.9
- net ~{FAULT_ISO}: now also J7.12; no longer J7.7
- net ~{READY_ISO}: now also J7.14; no longer J7.5
Other:
- moved on the sheet: J3, J7, J8
